Commit message: Adjusted the robotic manipulator URDF and added some collision tags

File: src/robotic_arm_description/urdf/robotic_arm.xacro (robot description, xacro)
@@ -1,4 +1,4 @@
 <?xml version="1.0"?>
-<robot  name= "robotic_arm" xmlns:xacro="http://www.ros.org/wiki/xacro">
+<robot xmlns:xacro="http://www.ros.org/wiki/xacro">
     <link name = "base_link">
         <visual>
@@ -6,9 +6,13 @@
                 <box size="0.4 0.4 0.1" />
             </geometry>
-            <origin xyz = "0 0 0" rpy = "0 0 0" />
-            <material name="grey">
-                <color rgba="0.5 0.5 0.5 1" />
-            </material>
+            <origin xyz = "0 0 0.05" rpy = "0 0 0" />
+            <material name="grey"/>
         </visual>
+        <collision>
+            <geometry>
+                <box size="0.4 0.4 0.1" />
+            </geometry>
+            <origin xyz = "0 0 0.05" rpy = "0 0 0" />
+        </collision>
     </link>
     <link name = "shoulder_link">
@@ -17,9 +21,13 @@
                 <cylinder radius="0.1" length="0.5" />
             </geometry>
-            <origin xyz = "0 0 0" rpy = "0 0 0" />
-            <material name="blue">
-               <color rgba="0 0 0.5 1" />
-            </material>
+            <origin xyz = "0 0 0.25" rpy = "0 0 0" />
+            <material name="blue"/>
         </visual>
+        <collision>
+            <geometry>
+                <box size="0.2 0.2 0.5" />
+            </geometry>
+            <origin xyz = "0 0 0.25" rpy = "0 0 0" />
+        </collision>
     </link>
     <link name = "arm_link">
@@ -29,8 +37,12 @@
             </geometry>
             <origin xyz = "0 0 0.3" rpy = "0 0 0" />
-            <material name="grey">
-                <color rgba="0.5 0.5 0.5 1" />
-            </material>
+            <material name="grey"/>
         </visual>
+        <collision>
+            <geometry>
+                <box size="0.1 0.1 0.6" />
+            </geometry>
+            <origin xyz = "0 0 0.3" rpy = "0 0 0" />
+        </collision>
     </link>
     <link name = "elbow_link" >
@@ -39,9 +51,13 @@
                 <cylinder radius="0.05" length="0.1" />
             </geometry>
-            <origin xyz = "0 0 0" rpy = "0 0 0" />
-            <material name="blue">
-               <color rgba="0 0 0.5 1" />
-            </material>
+            <origin xyz = "0 0 0.05" rpy = "0 0 0" />
+            <material name="blue"/>
         </visual>
+        <collision>
+            <geometry>
+                <box size="0.1 0.1 0.1" />
+            </geometry>
+            <origin xyz = "0 0 0.05" rpy = "0 0 0" />
+        </collision>
     </link>
     <link name = "forearm_link">
@@ -50,9 +66,13 @@
                 <cylinder radius="0.05" length="0.5" />
             </geometry>
-            <origin xyz = "0 0 0" rpy = "0 0 0" />
-            <material name="grey">
-                <color rgba="0.5 0.5 0.5 1" />
-            </material>
+            <origin xyz = "0 0 0.25" rpy = "0 0 0" />
+            <material name="grey"/>
         </visual>
+        <collision>
+            <geometry>
+                <box size="0.1 0.1 0.5" />
+            </geometry>
+            <origin xyz = "0 0 0.25" rpy = "0 0 0" />
+        </collision>
     </link>
     <link name = "wrist_link">
@@ -61,9 +81,13 @@
                 <box size= "0.1 0.1 0.05" />
             </geometry>
-            <origin xyz = "0 0 0" rpy = "0 0 0" />
-            <material name="blue">
-               <color rgba="0 0 0.5 1" />
-            </material>
+            <origin xyz = "0 0 0.025" rpy = "0 0 0" />
+            <material name="blue"/>
         </visual>
+        <collision>
+            <geometry>
+                <box size= "0.1 0.1 0.05" />
+            </geometry>
+            <origin xyz = "0 0 0.025" rpy = "0 0 0" />
+        </collision>
     </link>
     <link name = "hand_link">
@@ -72,23 +96,20 @@
                 <box size= "0.1 0.1 0.02" />
             </geometry>
-            <origin xyz = "0 0 0" rpy = "0 0 0" />
-            <material name="grey">
-                <color rgba="0.5 0.5 0.5 1" />
-            </material>
+            <origin xyz = "0 0 0.01" rpy = "0 0 0" />
+            <material name="grey"/>
         </visual>
+        <collision>
+            <geometry>
+                <box size= "0.1 0.1 0.05" />
+            </geometry>
+            <origin xyz = "0 0 0.025" rpy = "0 0 0" />
+        </collision>
     </link>
     <link name = "tool_link">
     </link>
-    <link name = "root_link">
-    </link>
-    <joint name = "root_bae_joint" type = "fixed">
-        <parent link =  "root_link" />
-        <child link = "base_link" />
-        <origin xyz  = "0 0 0.05" rpy="0 0 0"/>
-    </joint>
     <joint name = "base_shoulder_joint" type = "revolute">
         <parent link =  "base_link" />
         <child link = "shoulder_link" />
-        <origin xyz  = "0 0 0.3" rpy="0 0 0"/>
+        <origin xyz  = "0 0 0.1" rpy="0 0 0"/>
         <axis xyz = "0 0 1" />
         <limit effort= "1000.0" velocity="1.0" lower= "-3.14" upper= "3.14" />
@@ -97,5 +118,5 @@
         <parent link =  "shoulder_link" />
         <child link = "arm_link" />
-        <origin xyz  = "0 0 0.25" rpy="0 0 0"/>
+        <origin xyz  = "0 0 0.5" rpy="0 0 0"/>
         <axis xyz = "0 1 0" />
         <limit effort= "1000.0" velocity="1.0" lower= "0" upper= "2.5" />
@@ -104,5 +125,5 @@
         <parent link =  "arm_link" />
         <child link = "elbow_link" />
-        <origin xyz  = "0 0 0.65" rpy="0 0 0"/>
+        <origin xyz  = "0 0 0.6" rpy="0 0 0"/>
         <axis xyz = "0 1 0" />
         <limit effort= "1000.0" velocity="1.0" lower= "0" upper= "2.5" />
@@ -111,5 +132,5 @@
         <parent link =  "elbow_link" />
         <child link = "forearm_link" />
-        <origin xyz  = "0 0 0.3" rpy="0 0 0"/>
+        <origin xyz  = "0 0 0.1" rpy="0 0 0"/>
         <axis xyz = "0 0 1" />
         <limit effort= "1000.0" velocity="1.0" lower= "-3.14" upper= "3.14" />
@@ -118,5 +139,5 @@
         <parent link =  "forearm_link" />
         <child link = "wrist_link" />
-        <origin xyz  = "0 0 0.275" rpy="0 0 0"/>
+        <origin xyz  = "0 0 0.5" rpy="0 0 0"/>
         <axis xyz = "0 1 0" />
         <limit effort= "1000.0" velocity="1.0" lower= "-1.57" upper= "1.57" />
@@ -125,5 +146,5 @@
         <parent link =  "wrist_link" />
         <child link = "hand_link" />
-        <origin xyz  = "0 0 0.035" rpy="0 0 0"/>
+        <origin xyz  = "0 0 0.05" rpy="0 0 0"/>
         <axis xyz = "0 0 1" />
     </joint>
