Commit message: configued moveit for the robot

File: src/robotic_arm_description/urdf/common_properties.xacro (robot description, xacro)
@@ -1,4 +1,4 @@
 <?xml version="1.0"?>
-<robot name= "robotic_arm" xmlns:xacro="http://www.ros.org/wiki/xacro">
+<robot xmlns:xacro="http://www.ros.org/wiki/xacro">
     <material name="grey">
         <color rgba="0.5 0.5 0.5 1" />
@@ -7,3 +7,9 @@
         <color rgba="0 0 0.5 1" />
     </material>
+    <material name="dark_green">
+        <color rgba="0 0.4 0 1" />
+    </material>
+    <material name="light_green">
+        <color rgba="0 0.6 0 1" />
+    </material>
 </robot>

File: src/robotic_arm_description/urdf/main_robotic_arm.urdf.xacro (robot description, xacro)
@@ -3,3 +3,9 @@
    <xacro:include filename="common_properties.xacro" />
    <xacro:include filename="robotic_arm.xacro" />
+   <xacro:include filename="gripper.xacro" />
+   <joint name="arm_gripper_joint" type="fixed">
+      <parent link="tool_link" />
+      <child link="gripper_base_link" />
+      <origin xyz="0 0 0" rpy="0 0 0" />
+   </joint>
 </robot>

File: src/robotic_arm_description/urdf/robotic_arm.xacro (robot description, xacro)
@@ -101,7 +101,7 @@
         <collision>
             <geometry>
-                <box size= "0.1 0.1 0.05" />
+                <box size= "0.1 0.1 0.02" />
             </geometry>
-            <origin xyz = "0 0 0.025" rpy = "0 0 0" />
+            <origin xyz = "0 0 0.01" rpy = "0 0 0" />
         </collision>
     </link>
@@ -152,5 +152,5 @@
         <parent link =  "hand_link" />
         <child link = "tool_link" />
-        <origin xyz  = "0 0 0" rpy="0 0 0"/>
+        <origin xyz  = "0 0 0.02" rpy="0 0 0"/>
     </joint>
 </robot>

File: src/robotic_arm_moveit_config/config/robotic_arm.ros2_control.xacro (robot description, xacro)
@@ -44,4 +44,10 @@
                 </state_interface>
             </joint>
+            <joint name="gripper_base_left_joint">
+                <command_interface name="position"/>
+                <state_interface name="position">
+                  <param name="initial_value">${initial_positions['gripper_base_left_joint']}</param>
+                </state_interface>
+            </joint>
         </ros2_control>
     </xacro:macro>
